Commit message: updated humanoid urdf, disabled viewer camera lock on vis robot motions

File: GMR_Wato/humanoid_urdf/pioneer_humanoid.urdf (robot description, URDF)
Before this commit: robot pioneer_humanoid, 68 links, 67 joints
Links:
- added link head, mass 0.2599; collision box size=0.178958 0.201527 0.242703; visual mesh filename=meshes/head_0.obj scale=0.001 0.001 0.001
- added link neck_link, mass 0.1074; collision box size=0.185918 0.169320 0.196946; visual mesh filename=meshes/neck_link_0.obj scale=0.001 0.001 0.001
- link l_foot: mass 0.2889 -> 0.1497; geometry collision box size=0.114000 0.243131 0.084400; visual mesh filename=meshes/l_foot_0.obj scale=0.001 0.001 0.001
- link l_shank_foot: mass 0.4385 -> 0.4730; geometry collision box size=0.115500 0.118992 0.469596; visual mesh filename=meshes/l_shank_foot_0.obj scale=0.001 0.001 0.001
- link l_thigh: mass 0.9437 -> 0.9705
- link torso: mass 1.4254 -> 1.2415; geometry collision box size=0.326650 0.293938 0.488000; visual mesh filename=meshes/torso_0.obj scale=0.001 0.001 0.001
Joints:
- added joint neck_pitch: type revolute, parent neck_link, child head, origin xyz=0.000000 0.000000 0.196946, axis 1.000000 0.000000 0.000000, limit lower=-0.3491 upper=0.5236 effort=10 velocity=6
- added joint neck_yaw: type revolute, parent torso, child neck_link, origin xyz=0.000000 0.000000 0.364000, axis 0.000000 0.000000 1.000000, limit lower=-1.2217 upper=1.2217 effort=10 velocity=6
- joint Ankle_P_R: axis -1.000000 0.000000 0.000000 -> 1.000000 0.000000 0.000000
- joint Ankle_R_L: limit lower=-0.5236 upper=0.5236 effort=10 velocity=6 -> lower=-0.2618 upper=0.2618 effort=10 velocity=6
- joint Ankle_R_R: limit lower=-0.5236 upper=0.5236 effort=10 velocity=6 -> lower=-0.2618 upper=0.2618 effort=10 velocity=6
- joint Hip_A_L: axis 0.000000 1.000000 0.000000 -> 0.000000 -1.000000 0.000000
- joint Knee_L: limit lower=-1.0472 upper=0.0873 effort=10 velocity=6 -> lower=-1.1345 upper=0.0 effort=10 velocity=6
- joint Knee_R: limit lower=-1.0472 upper=0.0873 effort=10 velocity=6 -> lower=-1.1345 upper=0.0 effort=10 velocity=6

File: GMR_Wato/humanoid_urdf/pioneer_humanoid_mujoco.urdf (robot description, URDF)
Before this commit: robot pioneer_humanoid, 68 links, 67 joints
Links:
- added link head, mass 0.2599; collision box size=0.178958 0.201527 0.242703; visual mesh filename=meshes/head_0.obj scale=0.001 0.001 0.001
- added link neck_link, mass 0.1074; collision box size=0.185918 0.169320 0.196946; visual mesh filename=meshes/neck_link_0.obj scale=0.001 0.001 0.001
- link l_foot: mass 0.2889 -> 0.1497; geometry collision box size=0.114000 0.243131 0.084400; visual mesh filename=meshes/l_foot_0.obj scale=0.001 0.001 0.001
- link l_shank_foot: mass 0.4385 -> 0.4730; geometry collision box size=0.115500 0.118992 0.469596; visual mesh filename=meshes/l_shank_foot_0.obj scale=0.001 0.001 0.001
- link l_thigh: mass 0.9437 -> 0.9705
- link torso: mass 1.4254 -> 1.2415; geometry collision box size=0.326650 0.293938 0.488000; visual mesh filename=meshes/torso_0.obj scale=0.001 0.001 0.001
Joints:
- added joint neck_pitch: type revolute, parent neck_link, child head, origin xyz=0.000000 0.000000 0.196946, axis 1.000000 0.000000 0.000000, limit lower=-0.3491 upper=0.5236 effort=10 velocity=6
- added joint neck_yaw: type revolute, parent torso, child neck_link, origin xyz=0.000000 0.000000 0.364000, axis 0.000000 0.000000 1.000000, limit lower=-1.2217 upper=1.2217 effort=10 velocity=6
- joint Ankle_P_R: axis -1.000000 0.000000 0.000000 -> 1.000000 0.000000 0.000000
- joint Ankle_R_L: limit lower=-0.5236 upper=0.5236 effort=10 velocity=6 -> lower=-0.2618 upper=0.2618 effort=10 velocity=6
- joint Ankle_R_R: limit lower=-0.5236 upper=0.5236 effort=10 velocity=6 -> lower=-0.2618 upper=0.2618 effort=10 velocity=6
- joint Hip_A_L: axis 0.000000 1.000000 0.000000 -> 0.000000 -1.000000 0.000000
- joint Knee_L: limit lower=-1.0472 upper=0.0873 effort=10 velocity=6 -> lower=-1.1345 upper=0.0 effort=10 velocity=6
- joint Knee_R: limit lower=-1.0472 upper=0.0873 effort=10 velocity=6 -> lower=-1.1345 upper=0.0 effort=10 velocity=6
